Commit message: Prepare the Pioneer 3AT for off-board slam_toolbox
- drive: publish the yaw rate in twist.angular.z (it went to angular.x)
  and fill diagonal odometry covariances
- description: set the measured BNO055 stick mounting rotation
- bringup: add slam_sensors.launch.py with the robot description, Aria,
  SICK LMS 200 and IMU drivers

Co-Authored-By: Claude Opus 5.5 <noreply@anthropic.com>

File: pioneer_description/urdf/pioneer3at_calibration.xacro (robot description, xacro)
@@ -91,10 +91,12 @@
   <xacro:property name="gps_rot_y" value="0.0" />
   <xacro:property name="gps_rot_z" value="0.0" />
-  <!-- IMU -->
+  <!-- IMU: BNO055 USB stick standing with its USB-A connector down, sensor +x facing
+       left and +z facing backward. Rotation measured from gravity and lidar scan
+       matching on 2026-10-20; the stick's position barely matters for a gyro. -->
   <xacro:property name="imu_trans_x" value="0.0" />
   <xacro:property name="imu_trans_y" value="-0.10" />
   <xacro:property name="imu_trans_z" value="0.0" />
-  <xacro:property name="imu_rot_x" value="0.0" />
-  <xacro:property name="imu_rot_y" value="0.0" />
-  <xacro:property name="imu_rot_z" value="0.0" />
+  <xacro:property name="imu_rot_x" value="-1.5179" />
+  <xacro:property name="imu_rot_y" value="0.0110" />
+  <xacro:property name="imu_rot_z" value="1.5714" />
 </robot>

Commit message: Set the measured SICK LMS 200 mounting position
Scan plane 0.34 m above the floor, 0.125 m ahead of the robot center.

Co-Authored-By: Claude Opus 5.5 <noreply@anthropic.com>

File: pioneer_description/urdf/pioneer3at_calibration.xacro (robot description, xacro)
@@ -28,8 +28,10 @@
   <xacro:property name="footprint_rot_y" value="0.0" />
   <xacro:property name="footprint_rot_z" value="0.0" />
-  <!-- Top laser (base_laser_link) -->
+  <!-- Top laser (base_laser_link), relative to lidar_support. The SICK LMS 200 faces
+       forward with its scan plane 0.34 m above the floor and 0.125 m ahead of the robot
+       center (measured 2026-10-20); top_plate is at z = 0.274. -->
   <xacro:property name="top_laser_trans_x" value="0.0" />
   <xacro:property name="top_laser_trans_y" value="0.0" />
-  <xacro:property name="top_laser_trans_z" value="0.23" />
+  <xacro:property name="top_laser_trans_z" value="0.066" />
   <xacro:property name="top_laser_rot_x" value="0.0" />
   <xacro:property name="top_laser_rot_y" value="0.0" />
@@ -71,5 +73,5 @@
   <xacro:property name="back_right_axle_trans_z" value="0.111" />
   <!-- Top Laser Support (lidar support) -->
-  <xacro:property name="top_laser_support_trans_x" value="-0.07" />
+  <xacro:property name="top_laser_support_trans_x" value="0.122" />
   <xacro:property name="top_laser_support_trans_y" value="0.0" />
   <xacro:property name="top_laser_support_trans_z" value="0.0" />
